Commit message: Update robot description and world assets

File: description/gazebo_control.xacro (robot description, xacro)
@@ -5,5 +5,5 @@
             <!--Wheel Information-->
             <left_joint>left_wheel_joint</left_joint>
-            <right_joint>left_wheel_joint</right_joint>
+            <right_joint>right_wheel_joint</right_joint>
             <wheel_separation>0.35</wheel_separation>
             <wheel_diameter>0.1</wheel_diameter>
@@ -16,5 +16,5 @@
             <publish_odom>true</publish_odom>
             <publish_odom_tf>true</publish_odom_tf>
-            <pulblish_wheel_tf>true</pulblish_wheel_tf>
+            <publish_wheel_tf>true</publish_wheel_tf>
         </plugin>
     </gazebo>

File: description/robot_core.xacro (robot description, xacro)
@@ -13,4 +13,7 @@
     <material name="black">
         <color rgba="0 0 0 1"/>
+    </material>
+    <material name="red">
+        <color rgba="1 0 0 1"/>
     </material>
     <!--Base link-->
